File: bored27-revision.kicad_sch (KiCad schematic)
At the start: 19 parts, among them J1 USB_C_Receptacle_USB2.0, J2 AVR-ISP-6, SW1 SW_Push, U1 ATmega32U2-A, U2 PRTR5V0U2X, X1 16MHz

Commit message: finished pcb
Parts:
- added FB1: 60@100MHz, Inductor_SMD:L_0805_2012Metric_Pad1.15x1.40mm_HandSolder, symbol Device:FerriteBead_Small
Connections:
- net COL0: now also U1.22 (PC7); no longer U1.21 (PB7)
- net COL1: now also U1.21 (PB7); no longer U1.5 (PC2)
- net COL2: now also U1.20 (PB6); no longer U1.26 (PC4)
- net COL3: now also U1.19 (PB5); no longer U1.25 (PC5)
- net COL4: now also U1.26 (PC4); no longer U1.23 (PC6)
- net COL5: now also U1.18 (PB4); no longer U1.22 (PC7)
- net COL6: now also U1.11 (PD5); no longer U1.6 (PD0)
- net COL7: now also U1.9 (PD3); no longer U1.7 (PD1)
- net COL8: now also U1.7 (PD1); no longer U1.8 (PD2)
- net COL9: now also U1.5 (PC2); no longer U1.9 (PD3)
- net D+: now also R3.2, U1.29 (D+); no longer J1.A6 (D+), J1.B6 (D+), R3.1, U2.2 (IO1)
- net D-: now also R4.2, U1.30 (D-); no longer J1.A7 (D-), J1.B7 (D-), R4.1, U2.3 (IO2)
- net GND: now also FB1.2; no longer J1.S1 (SHIELD)
- net ROW0: now also U1.6 (PD0); no longer U1.14 (PB0)
- net ROW1: now also U1.8 (PD2); no longer U1.18 (PB4)
- net ROW2: now also U1.10 (PD4); no longer U1.19 (PB5)
- net ROW3: now also U1.25 (PC5); no longer U1.20 (PB6)
- new net DN: J1.A7 (D-), J1.B7 (D-), R4.1, U2.3 (IO2)
- new net DP: J1.A6 (D+), J1.B6 (D+), R3.1, U2.2 (IO1)
- new net Earth: FB1.1, J1.S1 (SHIELD)
Other:
- note added: "usb-c&esd"
- note removed: "esd"
- note removed: "usb-c"
- moved on the sheet: R3, R4, U2
